File: hellen64_NB1.kicad_pcb (KiCad board)
At the start: 2 copper layers, 154 x 159 mm, 168 parts, among them J1 USB_B_Mini, J11 Conn_01x01, J13 Conn_01x01, J14 Conn_01x01, J15 Conn_01x01, J16 Conn_01x01, J17 Conn_01x01, J19 Conn_01x01, J2 Conn_01x05_Male, J20 Conn_01x01, J21 Conn_01x01, J22 Conn_01x01, J24 Conn_01x01, J25 AudioJack3_SwitchTR, J27 Conn_01x06, J4 Conn_02x12_Odd_Even, J5 USB_B, M1 Module-input-0.1, M10 Module-power12-0.2, M11 Module-power5-0.2, M12 Module-wbo-0.2, M13 Module-can-0.1, M2 Module-ign8-0.1, M3 Module-mcu-0.3, M4 Module-sd-0.1, M5 Module-output-0.2, M6 Module-dinput4-0.1, M7 Module-stlink-0.1, M8 Module-can-0.1, M9 Module-knock-0.1, P1 Pad, P10 Pad, P11 Pad, P12 Pad, P13 Pad, P14 Pad, P15 Pad, P17 Pad, P18 Pad, P19 Pad, P2 178780-1, P20 Pad, P22 Pad, P23 Pad, P24 Pad, P25 Pad, P27 Pad, P28 Pad, P29 Pad, P3 Pad, P30 Pad, P31 Pad, P32 Pad, P34 Pad, P38 Pad, P4 Pad, P43 Pad, P44 Pad, P46 Pad, P47 Pad, P48 Pad, P49 Pad, P5 Pad, P50 Pad, P51 Pad, P52 Pad, P53 Pad, P55 Pad, P56 Pad, P6 Pad, P7 Pad, P8 Pad, P9 Pad, U1 LIS2DW12TR, U2 MPX4_MAP, U3 MCP6002-xSN, U4 LPS25HB

Commit message: update
Parts:
- removed P27, P46: Pad, hellen-one-common:PAD-TH
- added C10: 10nF, hellen-one-common:C0603, F.Cu at (63.3, 70.1)
- added C11: 10uF, hellen-one-common:C0805, F.Cu at (59.2, 50.9)
- added C12: 10uF, hellen-one-common:C0805, F.Cu at (60.7, 50.9)
- added C13: 10uF, hellen-one-common:C0805, F.Cu at (62.2, 50.9)
- added C14: 220nF, hellen-one-common:C0603, F.Cu at (57.0, 54.4)
- added C15: 10uF, hellen-one-common:C0805, F.Cu at (63.7, 50.9)
- added C16: 10uF, hellen-one-common:C0805, F.Cu at (65.2, 50.9)
- added C17: 10uF, hellen-one-common:C0805, F.Cu at (66.7, 50.9)
- added C18: 10uF, hellen-one-common:C0805, F.Cu at (68.2, 50.9)
- added C19: 10uF, hellen-one-common:C0805, F.Cu at (69.7, 50.9)
- added C20: 10uF, hellen-one-common:C0805, F.Cu at (71.2, 50.9)
- added C7: 100nF, hellen-one-common:C0603, F.Cu at (56.2, 51.2)
- added C8: 6.8nF, hellen-one-common:C0603, F.Cu at (66.0, 70.1)
- added C9: 10uF, hellen-one-common:C0805, F.Cu at (57.7, 50.9)
- added D33: 1N4148WS, hellen-one-common:SOD-323, F.Cu at (60.1, 72.6)
- added D34: 1N4148WS, hellen-one-common:SOD-323, F.Cu at (63.4, 72.6)
- added F3: Fuse-Pad-Pad, hellen-one-common:PAD-1206-PAD, F.Cu at (44.7, 35.9)
- added J3: MiniFit, hellen-one-common:Molex-39301020, F.Cu at (48.5, 69.2)
- added J6: ETB, hellen-one-common:PinHeader_1x06_P2.54mm_Vertical, F.Cu at (75.0, 64.5)
- added R10: 100, hellen-one-common:R0603, F.Cu at (63.3, 71.4)
- added R19: 10k, hellen-one-common:R0603, F.Cu at (66.7, 72.6)
- added R21: Jumper-Pad-Pad, hellen-one-common:PAD-0805-PAD, F.Cu at (77.1, 41.7)
- added R22: Jumper-Pad-Pad, hellen-one-common:PAD-0805-PAD, F.Cu at (62.6, 41.7)
- added R9: 100k, hellen-one-common:R0603, F.Cu at (65.9, 71.3)
- added U5: L6205PD, hellen-one-common:SO20POWER, F.Cu at (64.8, 61.5)
- moved P56 62.4 mm to (63.3, 37.0)
- moved R20 20.0 mm to (58.0, 41.5)
- moved D11 13.8 mm to (49.5, 80.8)
- moved D5 13.8 mm to (47.6, 80.8)
- moved R2 13.8 mm to (46.2, 84.7)
- moved R5 13.8 mm to (48.7, 84.7)
- moved D10 13.8 mm to (45.8, 80.9)
- moved P47 10.0 mm to (55.5, 37.3)
- moved R40 6.70 mm to (44.2, 42.5)
- moved M11 5.61 mm to (42.8, 113.0)
- moved G4 4.99 mm to (41.3, 125.6)
- moved G6 4.99 mm to (26.1, 125.6)
- moved R37 2.33 mm to (41.9, 42.5)
- moved R38 2.33 mm to (37.6, 42.5)
- moved R39 2.33 mm to (39.7, 42.5)
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Connections:
- net /LOW11 renamed /ALT_WARN
- net /SOLENOID_A1 renamed /ETB_EN
- net /SOLENOID_A2 renamed /+ETB
- net /SOLENOID_B1 renamed /-ETB
- net /WBO_H- renamed /4K
- M1 pad S4: /IN_NEUTRAL -> /IN_TPS2
- M5 pad S13: unconnected-(M5-PadS13) -> /OUT_ALT_WARNING
- M6 pad J2: GND -> +5V
- M6 pad J3: GND -> +5V
- M6 pad V4: /IN_D3 -> /IN_NEUTRAL
- P2 pad 66: /IN_TEMP -> Net-(P2-Pad66)
Routing:
- net /USB-: track 0.00 -> 393.3 mm, vias 0 -> 12
- net /USB+: track 393.3 -> 0.00 mm, vias 12 -> 0
- net /OUT_IGN1: track 545.7 -> 221.6 mm, vias 2 -> 1
- net /OUT_IGN2: track 1.54 -> 230.8 mm, vias 0 -> 1
- net /4K: track 226.1 -> 10.7 mm, vias 6 -> 0
- net /IN_CAM: track 477.9 -> 281.2 mm, vias 5 -> 3
- net +5VA: track 378.2 -> 251.8 mm, vias 14 -> 10
- net /IN_AFR: track 0.00 -> 95.2 mm, vias 0 -> 3
- net /IN_CLT: track 83.1 -> 5.56 mm, vias 2 -> 0
- net +12V_RAW: track 96.3 -> 169.9 mm, vias 3 -> 4
- net /OUT_TACH: track 73.4 -> 0.00 mm, vias 3 -> 0
- net /OUT_CHECK_ENGINE: track 70.0 -> 0.00 mm, vias 5 -> 0
- net /IN_PRESSURE: track 6.22 -> 72.7 mm, vias 0 -> 3
- net /OUT_VICS: track 0.00 -> 64.3 mm, vias 0 -> 1
- net /OUT_ECF: track 82.8 -> 23.7 mm
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
Commit message: update
Parts:
- moved P15 72.1 mm to (112.5, 37.0)
- moved P9 71.9 mm to (115.4, 37.0)
- moved P10 69.4 mm to (112.5, 40.0)
- moved R43 69.4 mm to (74.5, 41.0)
- moved P48 28.6 mm to (56.0, 37.0)
- moved R30 24.6 mm to (55.8, 41.0)
- moved R28 16.4 mm to (66.9, 41.0)
- moved R31 14.3 mm to (151.0, 48.2)
- moved R27 12.7 mm to (128.6, 41.5)
- moved P49 12.5 mm to (58.5, 46.1)
- moved P51 12.4 mm to (54.4, 46.1)
- moved P50 10.6 mm to (52.1, 37.0)
- moved P47 10.5 mm to (61.2, 46.1)
- moved P55 8.78 mm to (137.1, 39.2)
- moved R48 7.52 mm to (134.2, 41.7)
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Connections:
- M1 pad S18: /IN_TEMP -> /IN_TEMP_OR_PPS2
Routing:
- net /IN_CAM: track 281.2 -> 17.9 mm
- net /USB-: track 393.3 -> 189.5 mm, vias 12 -> 6
- net /USB+: track 0.00 -> 194.3 mm, vias 0 -> 6
- net /OUT_PUMP_RELAY: track 134.9 -> 0.00 mm, vias 2 -> 0
- net /OUT_TACH: track 0.00 -> 126.4 mm, vias 0 -> 3
- net /OUT_PUMP: track 0.00 -> 125.6 mm, vias 0 -> 2
- net /OUT_IGN2: track 230.8 -> 114.8 mm
- net /OUT_IGN1: track 221.6 -> 111.8 mm
- net /IN_AFR: track 95.2 -> 0.00 mm, vias 3 -> 0
- net /IN_CRANK: track 147.0 -> 62.6 mm, vias 2 -> 1
- net /3N: track 95.4 -> 12.0 mm, vias 3 -> 0
- net /IN_DIGITAL: track 10.7 -> 93.0 mm
- net /IN_PRESSURE: track 72.7 -> 6.22 mm, vias 3 -> 0
- net +12V_PROT: track 141.8 -> 75.6 mm, vias 8 -> 4
- net /IN_IAT: track 0.00 -> 60.1 mm, vias 0 -> 2
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