File: hellen64_NB1.kicad_sch (KiCad schematic)
At the start: 191 parts, among them J1 USB_B_Mini, J11 Conn_01x01, J13 Conn_01x01, J14 Conn_01x01, J15 Conn_01x01, J16 Conn_01x01, J17 Conn_01x01, J19 Conn_01x01, J2 Conn_01x05_Male, J20 Conn_01x01, J21 Conn_01x01, J22 Conn_01x01, J24 Conn_01x01, J25 AudioJack3_SwitchTR, J27 Conn_01x06, J3 MiniFit, J4 Conn_02x12_Odd_Even, J5 USB_B, J6 ETB, M1 Module-input-0.1, M10 Module-power12-0.2, M11 Module-power5-0.2, M12 Module-wbo-0.2, M13 Module-can-0.1, M2 Module-ign8-0.1, M3 Module-mcu-0.3, M4 Module-sd-0.1, M5 Module-output-0.2, M6 Module-dinput4-0.1, M7 Module-stlink-0.1, M8 Module-can-0.1, M9 Module-knock-0.1, P1 Pad, P10 Pad, P11 Pad, P12 Pad, P13 Pad, P14 Pad, P15 Pad, P17 Pad, P18 Pad, P19 Pad, P2 178780-1, P20 Pad, P22 Pad, P23 Pad, P24 Pad, P25 Pad, P28 Pad, P29 Pad, P3 Pad, P30 Pad, P31 Pad, P32 Pad, P34 Pad, P38 Pad, P4 Pad, P43 Pad, P44 Pad, P47 Pad, P48 Pad, P49 Pad, P5 Pad, P50 Pad, P51 Pad, P52 Pad, P53 Pad, P55 Pad, P56 Pad, P6 Pad, P7 Pad, P8 Pad, P9 Pad, U1 LIS2DW12TR, U2 MPX4_MAP, U3 MCP6002-xSN, U4 LPS25HB, U5 L6205PD

Commit message: update
Connections:
- net IN_TEMP is gone; now on net IN_TEMP_OR_PPS2: M1.S18 (IN_AUX2)
Other:
- note added: "EGR_BOOST"
Changed lines of the file:
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@@
     (effects (font (size 1.27 1.27)) (justify right bottom))
+  )
+  (text "EGR_BOOST" (at 196.85 90.17 0)
+    (effects (font (size 1.27 1.27)) (justify left bottom))
   )
   (text "Bus types" (at 199.39 247.65 0)
@@
     (effects (font (size 1.27 1.27)) (justify right bottom))
   )
+  (label "IN_PRESSURE" (at 292.1 260.35 0)
+    (effects (font (size 1.27 1.27)) (justify left bottom))
+  )
+  (label "IN_TEMP_OR_PPS2" (at 292.1 262.89 0)
+    (effects (font (size 1.27 1.27)) (justify left bottom))
+  )
+  (label "IN_AC_SW" (at 292.1 265.43 0)
+    (effects (font (size 1.27 1.27)) (justify left bottom))
+  )
+  (label "IN_EGR_BOOST" (at 292.1 267.97 0)
+    (effects (font (size 1.27 1.27)) (justify left bottom))
+  )
   (label "IN_TEMP_OR_PPS2" (at 293.37 328.93 180)
     (effects (font (size 1.27 1.27)) (justify right bottom))
   )
-  (label "IN_PRESSURE" (at 294.64 260.35 0)
-    (effects (font (size 1.27 1.27)) (justify left bottom))
-  )
-  (label "IN_TEMP" (at 294.64 262.89 0)
-    (effects (font (size 1.27 1.27)) (justify left bottom))
-  )
   (label "OUT_IGN1" (at 295.91 71.12 0)
     (effects (font (size 1.27 1.27)) (justify left bottom))
@@
     (effects (font (size 1.27 1.27)) (justify left bottom))
   )
-  (label "IN_AC_SW" (at 303.53 265.43 180)
-    (effects (font (size 1.27 1.27)) (justify right bottom))
-  )
   (label "IN_D4" (at 303.53 300.99 180)
     (effects (font (size 1.27 1.27)) (justify right bottom))
@@
     (effects (font (size 1.27 1.27)) (justify right bottom))
   )
-  (label "IN_EGR_BOOST" (at 308.61 267.97 180)
-    (effects (font (size 1.27 1.27)) (justify right bottom))
-  )

Commit message: update
Parts:
- removed P34: Pad, hellen-one-common:PAD-TH, symbol hellen-one-common:Pad
Connections:
- net OUT_CE is gone; now on net OUT_CHECK_ENGINE: D16.2 (K), D20.2 (A)
- net OUT_ECF is gone; now on net OUT_ECF_RELAY: D19.2 (K), D23.2 (A)
- net OUT_PUMP is gone; now on net OUT_PUMP_RELAY: D17.2 (K), D21.2 (A)
Changed lines of the file:
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@@
     (stroke (width 0.1524) (type solid) (color 0 0 0 0))
   )
+  (bus_entry (at 275.59 222.25) (size -2.54 2.54)
+    (stroke (width 0.1524) (type solid) (color 0 0 0 0))
+  )
   (bus_entry (at 275.59 224.79) (size -2.54 2.54)
     (stroke (width 0.1524) (type solid) (color 0 0 0 0))
@@
     (stroke (width 0) (type solid) (color 0 0 0 0))
   )
+  (wire (pts (xy 275.59 222.25) (xy 309.88 222.25))
+    (stroke (width 0) (type solid) (color 0 0 0 0))
+  )
   (wire (pts (xy 275.59 224.79) (xy 309.88 224.79))
     (stroke (width 0) (type solid) (color 0 0 0 0))
@@
     (stroke (width 0) (type solid) (color 0 0 0 0))
   )
-  (wire (pts (xy 294.64 222.25) (xy 309.88 222.25))
-    (stroke (width 0) (type solid) (color 0 0 0 0))
-  )
   (wire (pts (xy 294.64 245.11) (xy 309.88 245.11))
     (stroke (width 0) (type solid) (color 0 0 0 0))
@@
     (effects (font (size 1.27 1.27)) (justify right bottom))
   )
-  (label "OUT_CE" (at 83.82 337.82 180)
+  (label "OUT_CHECK_ENGINE" (at 83.82 337.82 180)
     (effects (font (size 1.27 1.27)) (justify right bottom))
   )
-  (label "OUT_PUMP" (at 83.82 347.98 180)
+  (label "OUT_PUMP_RELAY" (at 83.82 347.98 180)
     (effects (font (size 1.27 1.27)) (justify right bottom))
   )
@@
     (effects (font (size 1.27 1.27)) (justify right bottom))
   )
-  (label "OUT_ECF" (at 83.82 368.3 180)
+  (label "OUT_ECF_RELAY" (at 83.82 368.3 180)
     (effects (font (size 1.27 1.27)) (justify right bottom))
   )
@@
     (pin "1")
   )
-  (symbol (lib_id "hellen-one-common:Pad") (at 289.56 222.25 0) (mirror y) (unit 1)
-    (in_bom yes) (on_board yes)
-    (property "Reference" "P34" (id 0) (at 285.75 222.25 0))
-    (property "Value" "Pad" (id 1) (at 289.56 224.79 0)
-      (effects (font (size 1.27 1.27)) hide)
-    )
-    (property "Footprint" "hellen-one-common:PAD-TH" (id 2) (at 289.56 226.06 0)
-      (effects (font (size 1.27 1.27)) hide)
-    )
-    (property "Datasheet" "~" (id 3) (at 289.56 222.25 0)
-      (effects (font (size 1.27 1.27)) hide)
-    )
-    (pin "1")
-  )
   (symbol (lib_id "hellen-one-common:Pad") (at 289.56 245.11 0) (mirror y) (unit 1)
     (in_bom yes) (on_board yes)
@@
       (reference "P32") (unit 1) (value "Pad") (footprint "hellen-one-common:PAD-TH")
     )
-    (path "/96eb6f5f-5a3c-44a3-a70c-f52cba3f6e8b"
-      (reference "P34") (unit 1) (value "Pad") (footprint "hellen-one-common:PAD-TH")
-    )
     (path "/a1ceb4d6-d412-4dc3-b899-3531d409f675"

Commit message: pcb pre-alpha is ready
Parts:
- D25, D28, D31, D32: value 1N4148WS -> B5819W; footprint hellen-one-common:SOD-323 -> hellen-one-common:SOD-123; LCSC C2128 -> C8598
Connections:
- net IN_O2S is gone; now on net IN_AFR: M1.S9 (IN_O2S), P2.24 (2C)
- net O2S is gone; now on net AFR: M1.N18 (O2S), M3.S16 (IN_O2S)
- net +5VA: no longer M1.J19 (PULL_TPS), M1.J23 (PULL_SENS4), M1.J9 (PULL_AUX2)
- net AFR: no longer M1.N4 (O2S2), M3.S30 (IN_O2S2)
- net GND: now also J1.6 (Shield), M1.J19 (PULL_TPS), M1.J23 (PULL_SENS4), M1.J9 (PULL_AUX2)
- net IN_AFR: no longer M1.S25 (IN_O2S2), P2.26 (2G)
- net IN_TPS2: now also M1.S25 (IN_O2S2); no longer M1.S4 (IN_SENS4)
- net NEUTRAL renamed SENS4
- new net IN_O2S3: M1.S4 (IN_SENS4), P2.26 (2G)
- new net TPS2: M1.N4 (O2S2), M3.S30 (IN_O2S2)
- no-connect marks 54 -> 53
