File: hellen64_NB1.kicad_sch (KiCad schematic)
At the start: 190 parts, among them J1 USB_B_Mini, J11 Conn_01x01, J13 Conn_01x01, J14 Conn_01x01, J15 Conn_01x01, J16 Conn_01x01, J17 Conn_01x01, J19 Conn_01x01, J2 Conn_01x05_Male, J20 Conn_01x01, J21 Conn_01x01, J22 Conn_01x01, J24 Conn_01x01, J25 AudioJack3_SwitchTR, J27 Conn_01x06, J3 MiniFit, J4 Conn_02x12_Odd_Even, J5 USB_B, J6 ETB, M1 Module-input-0.1, M10 Module-power12-0.2, M11 Module-power5-0.2, M12 Module-wbo-0.2, M13 Module-can-0.1, M2 Module-ign8-0.1, M3 Module-mcu-0.3, M4 Module-sd-0.1, M5 Module-output-0.2, M6 Module-dinput4-0.1, M7 Module-stlink-0.1, M8 Module-can-0.1, M9 Module-knock-0.1, P1 Pad, P10 Pad, P11 Pad, P12 Pad, P13 Pad, P14 Pad, P15 Pad, P17 Pad, P18 Pad, P19 Pad, P2 178780-1, P20 Pad, P22 Pad, P23 Pad, P24 Pad, P25 Pad, P28 Pad, P29 Pad, P3 Pad, P30 Pad, P31 Pad, P32 Pad, P38 Pad, P4 Pad, P43 Pad, P44 Pad, P47 Pad, P48 Pad, P49 Pad, P5 Pad, P50 Pad, P51 Pad, P52 Pad, P53 Pad, P55 Pad, P56 Pad, P6 Pad, P7 Pad, P8 Pad, P9 Pad, U1 LIS2DW12TR, U2 MPX4_MAP, U3 MCP6002-xSN, U4 LPS25HB, U5 L6205PD

Commit message: https://github.com/rusefi/hellen-NB1-issues/issues/6 https://github.com/rusefi/hellen-NB1-issues/issues/7
Parts:
- added G11, G12, G9: PROTO_AREA, hellen-one-common:PROTO_AREA, symbol hellen-one-common:PROTO_AREA
Connections:
- new net: G11.1, G11.11, G11.6
- new net: G11.10, G11.15, G11.5
- new net: G11.12, G11.2, G11.7
- new net: G11.13, G11.3, G11.8
- new net: G11.14, G11.4, G11.9
- new net: G12.1, G12.11, G12.6
- new net: G12.10, G12.15, G12.5
- new net: G12.12, G12.2, G12.7
- new net: G12.13, G12.3, G12.8
- new net: G12.14, G12.4, G12.9
- new net: G9.1, G9.11, G9.6
- new net: G9.10, G9.15, G9.5
- new net: G9.12, G9.2, G9.7
- new net: G9.13, G9.3, G9.8
- new net: G9.14, G9.4, G9.9
Changed lines of the file:
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@@
   (junction (at 386.08 127) (diameter 1.016) (color 0 0 0 0))
   (junction (at 388.62 129.54) (diameter 1.016) (color 0 0 0 0))
+  (junction (at 513.08 308.61) (diameter 1.016) (color 0 0 0 0))
+  (junction (at 514.35 275.59) (diameter 1.016) (color 0 0 0 0))
+  (junction (at 514.35 292.1) (diameter 1.016) (color 0 0 0 0))
   (junction (at 515.62 62.23) (diameter 1.016) (color 0 0 0 0))
   (junction (at 515.62 64.77) (diameter 1.016) (color 0 0 0 0))
@@
   (junction (at 519.43 101.6) (diameter 1.016) (color 0 0 0 0))
   (junction (at 519.43 104.14) (diameter 1.016) (color 0 0 0 0))
+  (junction (at 519.43 308.61) (diameter 1.016) (color 0 0 0 0))
+  (junction (at 520.7 275.59) (diameter 1.016) (color 0 0 0 0))
+  (junction (at 520.7 292.1) (diameter 1.016) (color 0 0 0 0))
   (junction (at 521.97 204.47) (diameter 1.016) (color 0 0 0 0))
+  (junction (at 525.78 308.61) (diameter 1.016) (color 0 0 0 0))
+  (junction (at 527.05 275.59) (diameter 1.016) (color 0 0 0 0))
+  (junction (at 527.05 292.1) (diameter 1.016) (color 0 0 0 0))
+  (junction (at 532.13 308.61) (diameter 1.016) (color 0 0 0 0))
+  (junction (at 533.4 275.59) (diameter 1.016) (color 0 0 0 0))
+  (junction (at 533.4 292.1) (diameter 1.016) (color 0 0 0 0))
+  (junction (at 538.48 308.61) (diameter 1.016) (color 0 0 0 0))
+  (junction (at 539.75 275.59) (diameter 1.016) (color 0 0 0 0))
+  (junction (at 539.75 292.1) (diameter 1.016) (color 0 0 0 0))
   (junction (at 548.64 275.59) (diameter 1.016) (color 0 0 0 0))
   (junction (at 548.64 292.1) (diameter 1.016) (color 0 0 0 0))
@@
     (stroke (width 0) (type solid) (color 0 0 0 0))
   )
+  (wire (pts (xy 513.08 304.8) (xy 513.08 308.61))
+    (stroke (width 0) (type solid) (color 0 0 0 0))
+  )
+  (wire (pts (xy 513.08 308.61) (xy 513.08 312.42))
+    (stroke (width 0) (type solid) (color 0 0 0 0))
+  )
+  (wire (pts (xy 514.35 271.78) (xy 514.35 275.59))
+    (stroke (width 0) (type solid) (color 0 0 0 0))
+  )
+  (wire (pts (xy 514.35 275.59) (xy 514.35 279.4))
+    (stroke (width 0) (type solid) (color 0 0 0 0))
+  )
+  (wire (pts (xy 514.35 288.29) (xy 514.35 292.1))
+    (stroke (width 0) (type solid) (color 0 0 0 0))
+  )
+  (wire (pts (xy 514.35 292.1) (xy 514.35 295.91))
+    (stroke (width 0) (type solid) (color 0 0 0 0))
+  )
   (wire (pts (xy 515.62 62.23) (xy 510.54 62.23))
     (stroke (width 0) (type solid) (color 0 0 0 0))
@@
     (stroke (width 0) (type solid) (color 0 0 0 0))
   )
+  (wire (pts (xy 519.43 304.8) (xy 519.43 308.61))
+    (stroke (width 0) (type solid) (color 0 0 0 0))
+  )
+  (wire (pts (xy 519.43 308.61) (xy 519.43 312.42))
+    (stroke (width 0) (type solid) (color 0 0 0 0))
+  )
+  (wire (pts (xy 520.7 271.78) (xy 520.7 275.59))
+    (stroke (width 0) (type solid) (color 0 0 0 0))
+  )
+  (wire (pts (xy 520.7 275.59) (xy 520.7 279.4))
+    (stroke (width 0) (type solid) (color 0 0 0 0))
+  )
+  (wire (pts (xy 520.7 288.29) (xy 520.7 292.1))
+    (stroke (width 0) (type solid) (color 0 0 0 0))
+  )
+  (wire (pts (xy 520.7 292.1) (xy 520.7 295.91))
+    (stroke (width 0) (type solid) (color 0 0 0 0))
+  )
+  (wire (pts (xy 525.78 304.8) (xy 525.78 308.61))
+    (stroke (width 0) (type solid) (color 0 0 0 0))
+  )
+  (wire (pts (xy 525.78 308.61) (xy 525.78 312.42))
+    (stroke (width 0) (type solid) (color 0 0 0 0))
+  )
+  (wire (pts (xy 527.05 271.78) (xy 527.05 275.59))
+    (stroke (width 0) (type solid) (color 0 0 0 0))
+  )
+  (wire (pts (xy 527.05 275.59) (xy 527.05 279.4))
+    (stroke (width 0) (type solid) (color 0 0 0 0))
+  )
+  (wire (pts (xy 527.05 288.29) (xy 527.05 292.1))
+    (stroke (width 0) (type solid) (color 0 0 0 0))
+  )
+  (wire (pts (xy 527.05 292.1) (xy 527.05 295.91))
+    (stroke (width 0) (type solid) (color 0 0 0 0))
+  )
+  (wire (pts (xy 532.13 304.8) (xy 532.13 308.61))
+    (stroke (width 0) (type solid) (color 0 0 0 0))
+  )
+  (wire (pts (xy 532.13 308.61) (xy 532.13 312.42))
+    (stroke (width 0) (type solid) (color 0 0 0 0))
+  )
+  (wire (pts (xy 533.4 271.78) (xy 533.4 275.59))
+    (stroke (width 0) (type solid) (color 0 0 0 0))
+  )
+  (wire (pts (xy 533.4 275.59) (xy 533.4 279.4))
+    (stroke (width 0) (type solid) (color 0 0 0 0))
+  )
+  (wire (pts (xy 533.4 288.29) (xy 533.4 292.1))
+    (stroke (width 0) (type solid) (color 0 0 0 0))
+  )
+  (wire (pts (xy 533.4 292.1) (xy 533.4 295.91))
+    (stroke (width 0) (type solid) (color 0 0 0 0))
+  )
+  (wire (pts (xy 538.48 304.8) (xy 538.48 308.61))
+    (stroke (width 0) (type solid) (color 0 0 0 0))
+  )
+  (wire (pts (xy 538.48 308.61) (xy 538.48 312.42))
+    (stroke (width 0) (type solid) (color 0 0 0 0))
+  )
+  (wire (pts (xy 539.75 271.78) (xy 539.75 275.59))
+    (stroke (width 0) (type solid) (color 0 0 0 0))
+  )
+  (wire (pts (xy 539.75 275.59) (xy 539.75 279.4))
+    (stroke (width 0) (type solid) (color 0 0 0 0))
+  )
+  (wire (pts (xy 539.75 288.29) (xy 539.75 292.1))
+    (stroke (width 0) (type solid) (color 0 0 0 0))
+  )
+  (wire (pts (xy 539.75 292.1) (xy 539.75 295.91))
+    (stroke (width 0) (type solid) (color 0 0 0 0))
+  )
   (wire (pts (xy 548.64 271.78) (xy 548.64 275.59))
     (stroke (width 0) (type solid) (color 0 0 0 0))
@@
   (symbol (lib_id "power:GNDA") (at 354.33 339.09 90) (unit 1)
     (in_bom yes) (on_board yes)
-    (property "Reference" "#PWR?" (id 0) (at 360.68 339.09 0)
+    (property "Reference" "#PWR024" (id 0) (at 360.68 339.09 0)
       (effects (font (size 1.27 1.27)) hide)
     )
@@
     (pin "W5")
   )
+  (symbol (lib_id "hellen-one-common:PROTO_AREA") (at 539.75 304.8 0) (mirror y) (unit 1)
+    (in_bom yes) (on_board yes)
+    (property "Reference" "G9" (id 0) (at 538.48 300.99 0)
+      (effects (font (size 1.524 1.524)) hide)
+    )
+    (property "Value" "PROTO_AREA" (id 1) (at 522.5257 300.3482 0)
+      (effects (font (size 1.524 1.524)) (justify left))
+    )
+    (property "Footprint" "hellen-one-common:PROTO_AREA" (id 2) (at 524.51 316.23 0)
+      (effects (font (size 1.27 1.27)) hide)
+    )
+    (property "Datasheet" "" (id 3) (at 552.45 304.8 0)
+      (effects (font (size 1.27 1.27)) hide)
+    )
+    (pin "1")
+    (pin "10")
+    (pin "11")
+    (pin "12")
+    (pin "13")
+    (pin "14")
+    (pin "15")
+    (pin "2")
+    (pin "3")
+    (pin "4")
+    (pin "5")
+    (pin "6")
+    (pin "7")
+    (pin "8")
+    (pin "9")
+  )
+  (symbol (lib_id "hellen-one-common:PROTO_AREA") (at 541.02 271.78 0) (mirror y) (unit 1)
+    (in_bom yes) (on_board yes)
+    (property "Reference" "G11" (id 0) (at 539.75 267.97 0)
+      (effects (font (size 1.524 1.524)) hide)
+    )
+    (property "Value" "PROTO_AREA" (id 1) (at 523.7957 267.3282 0)
+      (effects (font (size 1.524 1.524)) (justify left))
+    )
+    (property "Footprint" "hellen-one-common:PROTO_AREA" (id 2) (at 525.78 283.21 0)
+      (effects (font (size 1.27 1.27)) hide)
+    )
+    (property "Datasheet" "" (id 3) (at 553.72 271.78 0)
+      (effects (font (size 1.27 1.27)) hide)
+    )
+    (pin "1")
+    (pin "10")
+    (pin "11")
+    (pin "12")
+    (pin "13")
+    (pin "14")
+    (pin "15")
+    (pin "2")
+    (pin "3")
+    (pin "4")
+    (pin "5")
+    (pin "6")
+    (pin "7")
+    (pin "8")
+    (pin "9")
+  )
+  (symbol (lib_id "hellen-one-common:PROTO_AREA") (at 541.02 288.29 0) (mirror y) (unit 1)
+    (in_bom yes) (on_board yes)
+    (property "Reference" "G12" (id 0) (at 539.75 284.48 0)
+      (effects (font (size 1.524 1.524)) hide)
+    )
+    (property "Value" "PROTO_AREA" (id 1) (at 523.7957 283.8382 0)
+      (effects (font (size 1.524 1.524)) (justify left))
+    )
+    (property "Footprint" "hellen-one-common:PROTO_AREA" (id 2) (at 525.78 299.72 0)
+      (effects (font (size 1.27 1.27)) hide)
+    )
+    (property "Datasheet" "" (id 3) (at 553.72 288.29 0)
+      (effects (font (size 1.27 1.27)) hide)
+    )
+    (pin "1")
+    (pin "10")
+    (pin "11")
+    (pin "12")
+    (pin "13")
+    (pin "14")
+    (pin "15")
+    (pin "2")
+    (pin "3")
+    (pin "4")
+    (pin "5")
+    (pin "6")
+    (pin "7")
+    (pin "8")
+    (pin "9")
+  )
   (symbol (lib_id "hellen-one-common:PROTO_AREA") (at 575.31 271.78 0) (mirror y) (unit 1)
     (in_bom yes) (on_board yes)
@@
       (reference "#PWR023") (unit 1) (value "+5VA") (footprint "")
     )
+    (path "/f8285b65-02a7-4092-88f9-49a6d6cb2309"
+      (reference "#PWR024") (unit 1) (value "GNDA") (footprint "")
+    )
     (path "/6552dfd4-22e7-4a28-99c4-ff2df27830e3"
       (reference "#PWR025") (unit 1) (value "GND") (footprint "")
@@
       (reference "#PWR0174") (unit 1) (value "+12V_PROT") (footprint "")
     )
-    (path "/f8285b65-02a7-4092-88f9-49a6d6cb2309"
-      (reference "#PWR?") (unit 1) (value "GNDA") (footprint "")
-    )
     (path "/b4512419-6564-4c85-97c7-af718c7ef6f7"
       (reference "BT1") (unit 1) (value "BATTERY_CR2032") (footprint "Battery:BatteryHolder_Keystone_1060_1x2032")
@@
       (reference "G7") (unit 1) (value "PROTO_AREA") (footprint "hellen-one-common:PROTO_AREA")
     )
+    (path "/ce3fd3d7-9d89-4db1-9f87-06dbd11bd511"
+      (reference "G9") (unit 1) (value "PROTO_AREA") (footprint "hellen-one-common:PROTO_AREA")
+    )
+    (path "/098fc9de-d2aa-4f8f-8d97-8427dcad36ff"
+      (reference "G11") (unit 1) (value "PROTO_AREA") (footprint "hellen-one-common:PROTO_AREA")
+    )
+    (path "/2cc47336-f714-4e64-82c3-84b9c5b7afbd"
+      (reference "G12") (unit 1) (value "PROTO_AREA") (footprint "hellen-one-common:PROTO_AREA")
+    )
     (path "/af907853-1b11-4836-8bf0-53e02c942215"

Commit message: update
Parts:
- C10: value 10nF -> 10n
- C11, C12, C13, C15, C16, C17, C18, C19, C20, C9: value 10uF -> 10u
- C14: value 220nF -> 220n
- C7: value 100nF -> 100n
- C8: value 6.8nF -> 6.8n
- M3: value Module-mcu-0.3 -> Module-mcu-0.5
Changed lines of the file:
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@@
       (effects (font (size 1.27 1.27)) (justify right))
     )
-    (property "Value" "100nF" (id 1) (at 217.8113 346.2021 90)
+    (property "Value" "100n" (id 1) (at 217.8113 346.2021 90)
       (effects (font (size 1.27 1.27)) (justify right))
     )
@@
       (effects (font (size 1.27 1.27)) (justify right))
     )
-    (property "Value" "10uF" (id 1) (at 226.9427 351.5359 90)
+    (property "Value" "10u" (id 1) (at 226.9427 351.5359 90)
       (effects (font (size 1.27 1.27)) (justify right))
     )
@@
       (effects (font (size 1.27 1.27)) (justify right))
     )
-    (property "Value" "6.8nF" (id 1) (at 226.0601 395.0907 90)
+    (property "Value" "6.8n" (id 1) (at 226.0601 395.0907 90)
       (effects (font (size 1.27 1.27)) (justify right))
     )
@@
       (effects (font (size 1.27 1.27)) (justify right))
     )
-    (property "Value" "10nF" (id 1) (at 234.6959 361.8293 90)
+    (property "Value" "10n" (id 1) (at 234.6959 361.8293 90)
       (effects (font (size 1.27 1.27)) (justify right))
     )
@@
       (effects (font (size 1.27 1.27)) (justify right))
     )
-    (property "Value" "10uF" (id 1) (at 235.8327 351.5359 90)
+    (property "Value" "10u" (id 1) (at 235.8327 351.5359 90)
       (effects (font (size 1.27 1.27)) (justify right))
     )
@@
       (effects (font (size 1.27 1.27)) (justify right))
     )
-    (property "Value" "10uF" (id 1) (at 244.7227 351.5359 90)
+    (property "Value" "10u" (id 1) (at 244.7227 351.5359 90)
       (effects (font (size 1.27 1.27)) (justify right))
     )
@@
       (effects (font (size 1.27 1.27)) (justify right))
     )
-    (property "Value" "10uF" (id 1) (at 253.6127 351.5359 90)
+    (property "Value" "10u" (id 1) (at 253.6127 351.5359 90)
       (effects (font (size 1.27 1.27)) (justify right))
     )
@@
       (effects (font (size 1.27 1.27)) (justify right))
     )
-    (property "Value" "220nF" (id 1) (at 256.1653 353.5681 90)
+    (property "Value" "220n" (id 1) (at 256.1653 353.5681 90)
       (effects (font (size 1.27 1.27)) (justify right))
     )
@@
       (effects (font (size 1.27 1.27)) (justify right))
     )
-    (property "Value" "10uF" (id 1) (at 262.5027 351.5359 90)
+    (property "Value" "10u" (id 1) (at 262.5027 351.5359 90)
       (effects (font (size 1.27 1.27)) (justify right))
     )
@@
       (effects (font (size 1.27 1.27)) (justify right))
     )
-    (property "Value" "10uF" (id 1) (at 270.1227 359.1559 90)
+    (property "Value" "10u" (id 1) (at 270.1227 359.1559 90)
       (effects (font (size 1.27 1.27)) (justify right))
     )
@@
       (effects (font (size 1.27 1.27)) (justify right))
     )
-    (property "Value" "10uF" (id 1) (at 271.3927 351.5359 90)
+    (property "Value" "10u" (id 1) (at 271.3927 351.5359 90)
       (effects (font (size 1.27 1.27)) (justify right))
     )
@@
       (effects (font (size 1.27 1.27)) (justify right))
     )
-    (property "Value" "10uF" (id 1) (at 280.2827 351.5359 90)
+    (property "Value" "10u" (id 1) (at 280.2827 351.5359 90)
       (effects (font (size 1.27 1.27)) (justify right))
     )
@@
       (effects (font (size 1.27 1.27)) (justify right))
     )
-    (property "Value" "10uF" (id 1) (at 280.2827 359.1559 90)
+    (property "Value" "10u" (id 1) (at 280.2827 359.1559 90)
       (effects (font (size 1.27 1.27)) (justify right))
     )
@@
       (effects (font (size 1.27 1.27)) (justify right))
     )
-    (property "Value" "10uF" (id 1) (at 290.4427 359.1559 90)
+    (property "Value" "10u" (id 1) (at 290.4427 359.1559 90)
       (effects (font (size 1.27 1.27)) (justify right))
     )
@@
     (in_bom yes) (on_board yes) (fields_autoplaced)
     (property "Reference" "M3" (id 0) (at 473.71 215.1338 0))
-    (property "Value" "Module-mcu-0.3" (id 1) (at 473.71 217.4325 0))
+    (property "Value" "Module-mcu-0.5" (id 1) (at 473.71 217.4325 0))
     (property "Footprint" "hellen-one-mcu-0.3:mcu" (id 2) (at 455.93 218.44 0)
       (effects (font (size 1.27 1.27)) hide)
@@
       (effects (font (size 1.27 1.27)) (justify left))
     )
-    (property "Value" "Module-mcu-0.3" (id 1) (at 418.4651 206.0078 0)
+    (property "Value" "Module-mcu-0.5" (id 1) (at 418.4651 206.0078 0)
       (effects (font (size 1.27 1.27)) (justify left))
     )
@@
       (effects (font (size 1.27 1.27)) (justify right))
     )
-    (property "Value" "Module-mcu-0.3" (id 1) (at 418.4651 67.5778 0)
+    (property "Value" "Module-mcu-0.5" (id 1) (at 418.4651 67.5778 0)
       (effects (font (size 1.27 1.27)) (justify right))
     )
@@
     (in_bom yes) (on_board yes) (fields_autoplaced)
     (property "Reference" "M3" (id 0) (at 445.9605 65.2738 0))
-    (property "Value" "Module-mcu-0.3" (id 1) (at 445.9605 67.5725 0))
+    (property "Value" "Module-mcu-0.5" (id 1) (at 445.9605 67.5725 0))
     (property "Footprint" "hellen-one-mcu-0.3:mcu" (id 2) (at 435.61 68.58 0)
       (effects (font (size 1.27 1.27)) hide)
@@
     )
     (path "/d1e13b8a-e2fb-4c9a-9728-ebeefa19c2ab"
-      (reference "C7") (unit 1) (value "100nF") (footprint "hellen-one-common:C0603")
+      (reference "C7") (unit 1) (value "100n") (footprint "hellen-one-common:C0603")
     )
     (path "/f9059228-1071-4ca2-914a-c0e8842bbc26"
-      (reference "C8") (unit 1) (value "6.8nF") (footprint "hellen-one-common:C0603")
+      (reference "C8") (unit 1) (value "6.8n") (footprint "hellen-one-common:C0603")
     )
     (path "/afabd0c1-3fc1-4838-9475-b9e6131c0bfc"
-      (reference "C9") (unit 1) (value "10uF") (footprint "hellen-one-common:C0805")
+      (reference "C9") (unit 1) (value "10u") (footprint "hellen-one-common:C0805")
     )
     (path "/e73d5392-969c-4bdc-8f49-bf64426a53cd"
-      (reference "C10") (unit 1) (value "10nF") (footprint "hellen-one-common:C0603")
+      (reference "C10") (unit 1) (value "10n") (footprint "hellen-one-common:C0603")
     )
     (path "/10a25306-9f13-4f92-947f-a107e99e7710"
-      (reference "C11") (unit 1) (value "10uF") (footprint "hellen-one-common:C0805")
+      (reference "C11") (unit 1) (value "10u") (footprint "hellen-one-common:C0805")
     )
     (path "/be8655a2-494b-40b4-98eb-293458785dcb"
-      (reference "C12") (unit 1) (value "10uF") (footprint "hellen-one-common:C0805")
+      (reference "C12") (unit 1) (value "10u") (footprint "hellen-one-common:C0805")
     )
     (path "/4c4fde36-9ed2-4cee-88c0-2e591d50821c"
-      (reference "C13") (unit 1) (value "10uF") (footprint "hellen-one-common:C0805")
+      (reference "C13") (unit 1) (value "10u") (footprint "hellen-one-common:C0805")
     )
     (path "/ebe21a06-e10e-47af-a5a4-58d6cea8761a"
-      (reference "C14") (unit 1) (value "220nF") (footprint "hellen-one-common:C0603")
+      (reference "C14") (unit 1) (value "220n") (footprint "hellen-one-common:C0603")
     )
     (path "/4ccd8695-6b1d-48ff-8fed-045eb0af7f79"
-      (reference "C15") (unit 1) (value "10uF") (footprint "hellen-one-common:C0805")
+      (reference "C15") (unit 1) (value "10u") (footprint "hellen-one-common:C0805")
     )
     (path "/992cb067-71f4-45b0-a273-7bcdd5313d63"
-      (reference "C16") (unit 1) (value "10uF") (footprint "hellen-one-common:C0805")
+      (reference "C16") (unit 1) (value "10u") (footprint "hellen-one-common:C0805")
     )
     (path "/30a68043-7bb6-45ef-9dab-59665482d70a"
-      (reference "C17") (unit 1) (value "10uF") (footprint "hellen-one-common:C0805")
+      (reference "C17") (unit 1) (value "10u") (footprint "hellen-one-common:C0805")
     )
     (path "/198d2042-fd0a-4b99-bb6a-e2e3e601b9e3"
-      (reference "C18") (unit 1) (value "10uF") (footprint "hellen-one-common:C0805")
+      (reference "C18") (unit 1) (value "10u") (footprint "hellen-one-common:C0805")
     )
     (path "/9a725c98-557d-42b7-8557-80e1e77fd8e5"
-      (reference "C19") (unit 1) (value "10uF") (footprint "hellen-one-common:C0805")
+      (reference "C19") (unit 1) (value "10u") (footprint "hellen-one-common:C0805")
     )
     (path "/8582dcf9-58d8-4236-a90f-8d632fa2f007"
-      (reference "C20") (unit 1) (value "10uF") (footprint "hellen-one-common:C0805")
+      (reference "C20") (unit 1) (value "10u") (footprint "hellen-one-common:C0805")
     )
     (path "/ecbba2ec-57c3-41e0-9e70-636da83aa612"
@@
     )
     (path "/a6bf355d-1d5f-4e79-8e3f-45e3bddf3ceb"
-      (reference "M3") (unit 1) (value "Module-mcu-0.3") (footprint "hellen-one-mcu-0.3:mcu")
+      (reference "M3") (unit 1) (value "Module-mcu-0.5") (footprint "hellen-one-mcu-0.3:mcu")
     )
     (path "/915d735b-9683-4d94-8b0d-1fa27ebac489"
-      (reference "M3") (unit 2) (value "Module-mcu-0.3") (footprint "hellen-one-mcu-0.3:mcu")
+      (reference "M3") (unit 2) (value "Module-mcu-0.5") (footprint "hellen-one-mcu-0.3:mcu")
     )
     (path "/5f1c7f30-e456-4e5e-847b-c87579bb1a4c"
-      (reference "M3") (unit 3) (value "Module-mcu-0.3") (footprint "hellen-one-mcu-0.3:mcu")
+      (reference "M3") (unit 3) (value "Module-mcu-0.5") (footprint "hellen-one-mcu-0.3:mcu")
     )
     (path "/a7d95f89-5755-415c-ab05-3cba0bcc1e6a"
-      (reference "M3") (unit 4) (value "Module-mcu-0.3") (footprint "hellen-one-mcu-0.3:mcu")
+      (reference "M3") (unit 4) (value "Module-mcu-0.5") (footprint "hellen-one-mcu-0.3:mcu")
     )
     (path "/46c92d79-ab77-4cea-933a-f95fdcee2757"
