File: hellen64_NB1.kicad_sch (KiCad schematic)
At the start: 193 parts, among them J1 USB_B_Mini, J11 Conn_01x01, J13 Conn_01x01, J14 Conn_01x01, J15 Conn_01x01, J16 Conn_01x01, J17 Conn_01x01, J19 Conn_01x01, J2 Conn_01x05_Male, J20 Conn_01x01, J21 Conn_01x01, J22 Conn_01x01, J24 Conn_01x01, J25 AudioJack3_SwitchTR, J27 Conn_01x06, J3 MiniFit, J4 Conn_02x12_Odd_Even, J5 USB_B, J6 ETB, M1 Module-input-0.1, M10 Module-power12-0.2, M11 Module-power5-0.2, M12 Module-wbo-0.2, M13 Module-can-0.1, M2 Module-ign8-0.1, M3 Module-mcu-0.5, M4 Module-sd-0.1, M5 Module-output-0.2, M6 Module-dinput4-0.1, M7 Module-stlink-0.1, M8 Module-can-0.1, M9 Module-knock-0.1, P1 Pad, P10 Pad, P11 Pad, P12 Pad, P13 Pad, P14 Pad, P15 Pad, P17 Pad, P18 Pad, P19 Pad, P2 178780-1, P20 Pad, P22 Pad, P23 Pad, P24 Pad, P25 Pad, P28 Pad, P29 Pad, P3 Pad, P30 Pad, P31 Pad, P32 Pad, P38 Pad, P4 Pad, P43 Pad, P44 Pad, P47 Pad, P48 Pad, P49 Pad, P5 Pad, P50 Pad, P51 Pad, P52 Pad, P53 Pad, P55 Pad, P56 Pad, P6 Pad, P7 Pad, P8 Pad, P9 Pad, U1 LIS2DW12TR, U2 MPX4_MAP, U3 MCP6002-xSN, U4 LPS25HB, U5 L6205PD

Commit message: fix AC_FAN_RELAY
Parts:
- removed P3: Pad, hellen-one-common:PAD-TH, symbol hellen-one-common:Pad
Connections:
- net IO7 is gone; now on net AC_FAN_RELAY: M3.E12 (OUT_IO2)
- net AC_FAN_RELAY: now reaches M5.W29 (LOW2)
- net ECF renamed ECF_RELAY
- net LOW1_DUAL renamed O2H
- net LOW2_DUAL renamed O2H2
- net LOW3_DUAL renamed MAIN
- net LOW5_HIGH1 renamed LOW7_HIGH1
- net LOW6_HIGH2 renamed AC_RELAY
- net LOW9 renamed LOW10
- net OUT_LOW3_DUAL renamed OUT_LOW5_DUAL
- net OUT_LOW5_PULLUP renamed OUT_LOW7_PULLUP
- net OUT_LOW9 renamed OUT_LOW10
- no-connect marks 53 -> 52
Changed lines of the file:
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@@
   (no_connect (at 354.33 326.39))
   (no_connect (at 354.33 336.55))
-  (no_connect (at 365.76 142.24))
   (no_connect (at 365.76 165.1))
   (no_connect (at 368.3 45.72))
@@
     (stroke (width 0) (type solid) (color 0 0 0 0))
   )
+  (wire (pts (xy 365.76 142.24) (xy 401.32 142.24))
+    (stroke (width 0) (type solid) (color 0 0 0 0))
+  )
   (wire (pts (xy 365.76 144.78) (xy 415.29 144.78))
     (stroke (width 0) (type solid) (color 0 0 0 0))
@@
     (stroke (width 0) (type solid) (color 0 0 0 0))
   )
+  (wire (pts (xy 401.32 147.32) (xy 401.32 142.24))
+    (stroke (width 0) (type solid) (color 0 0 0 0))
+  )
   (wire (pts (xy 414.02 20.32) (xy 419.1 20.32))
     (stroke (width 0) (type solid) (color 0 0 0 0))
@@
     (effects (font (size 1.27 1.27)) (justify right bottom))
   )
-  (label "OUT_LOW3_DUAL" (at 307.34 149.86 180)
+  (label "OUT_LOW5_DUAL" (at 307.34 149.86 180)
     (effects (font (size 1.27 1.27)) (justify right bottom))
   )
@@
     (effects (font (size 1.27 1.27)) (justify right bottom))
   )
-  (label "OUT_LOW5_PULLUP" (at 307.34 154.94 180)
+  (label "OUT_LOW7_PULLUP" (at 307.34 154.94 180)
     (effects (font (size 1.27 1.27)) (justify right bottom))
   )
@@
     (effects (font (size 1.27 1.27)) (justify right bottom))
   )
-  (label "OUT_LOW9" (at 307.34 162.56 180)
+  (label "OUT_LOW10" (at 307.34 162.56 180)
     (effects (font (size 1.27 1.27)) (justify right bottom))
   )
@@
     (effects (font (size 1.27 1.27)) (justify right bottom))
   )
-  (label "ECF" (at 378.46 139.7 180)
+  (label "ECF_RELAY" (at 378.46 139.7 180)
     (effects (font (size 1.27 1.27)) (justify right bottom))
   )
-  (label "LOW1_DUAL" (at 378.46 144.78 180)
+  (label "AC_FAN_RELAY" (at 378.46 142.24 180)
     (effects (font (size 1.27 1.27)) (justify right bottom))
   )
-  (label "LOW2_DUAL" (at 378.46 147.32 180)
+  (label "O2H" (at 378.46 144.78 180)
     (effects (font (size 1.27 1.27)) (justify right bottom))
   )
-  (label "LOW3_DUAL" (at 378.46 149.86 180)
+  (label "O2H2" (at 378.46 147.32 180)
+    (effects (font (size 1.27 1.27)) (justify right bottom))
+  )
+  (label "MAIN" (at 378.46 149.86 180)
     (effects (font (size 1.27 1.27)) (justify right bottom))
   )
@@
     (effects (font (size 1.27 1.27)) (justify right bottom))
   )
-  (label "LOW5_HIGH1" (at 378.46 154.94 180)
+  (label "LOW7_HIGH1" (at 378.46 154.94 180)
     (effects (font (size 1.27 1.27)) (justify right bottom))
   )
-  (label "LOW6_HIGH2" (at 378.46 157.48 180)
+  (label "AC_RELAY" (at 378.46 157.48 180)
     (effects (font (size 1.27 1.27)) (justify right bottom))
   )
@@
     (effects (font (size 1.27 1.27)) (justify right bottom))
   )
-  (label "LOW9" (at 378.46 162.56 180)
+  (label "LOW10" (at 378.46 162.56 180)
     (effects (font (size 1.27 1.27)) (justify right bottom))
   )
@@
     (effects (font (size 1.27 1.27)) (justify right bottom))
   )
-  (label "LOW2_DUAL" (at 414.02 165.1 180)
+  (label "O2H2" (at 414.02 165.1 180)
     (effects (font (size 1.27 1.27)) (justify right bottom))
   )
@@
     (pin "1")
   )
-  (symbol (lib_id "hellen-one-common:Pad") (at 396.24 147.32 180) (unit 1)
-    (in_bom yes) (on_board yes)
-    (property "Reference" "P3" (id 0) (at 393.7 147.32 0))
-    (property "Value" "Pad" (id 1) (at 396.24 144.78 0)
-      (effects (font (size 1.27 1.27)) hide)
-    )
-    (property "Footprint" "hellen-one-common:PAD-TH" (id 2) (at 396.24 143.51 0)
-      (effects (font (size 1.27 1.27)) hide)
-    )
-    (property "Datasheet" "~" (id 3) (at 396.24 147.32 0)
-      (effects (font (size 1.27 1.27)) hide)
-    )
-    (pin "1")
-  )
   (symbol (lib_id "hellen-one-common:Pad") (at 396.24 152.4 180) (unit 1)
     (in_bom yes) (on_board yes)
@@
       (reference "P2") (unit 4) (value "178780-1") (footprint "hellen-one-common:178780-1")
     )
-    (path "/6d0977fe-605a-4a9b-8286-b8b0b3b1cb58"
-      (reference "P3") (unit 1) (value "Pad") (footprint "hellen-one-common:PAD-TH")
-    )
     (path "/3bc39f4f-8a69-4179-86c7-4199afcc3826"

Commit message: JLC BOM adjustments
Parts:
- M3: value Module-mcu-0.5 -> Module-mcu144-0.5
Connections:
- net EXT_SPI_CS: now reaches M3.E4 (SPI1_CS1), U1.2 (~CS)
- net INJ5 renamed VVT
- net INJ6 renamed BOOST
- net INJ8 renamed VICS
Changed lines of the file:
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@@
     (effects (font (size 1.27 1.27)) (justify right bottom))
   )
-  (label "INJ1" (at 370.84 93.98 180)
+  (label "INJ1" (at 372.11 93.98 180)
     (effects (font (size 1.27 1.27)) (justify right bottom))
   )
-  (label "INJ2" (at 370.84 96.52 180)
+  (label "INJ2" (at 372.11 96.52 180)
     (effects (font (size 1.27 1.27)) (justify right bottom))
   )
-  (label "INJ3" (at 370.84 99.06 180)
+  (label "INJ3" (at 372.11 99.06 180)
     (effects (font (size 1.27 1.27)) (justify right bottom))
   )
-  (label "INJ4" (at 370.84 101.6 180)
+  (label "INJ4" (at 372.11 101.6 180)
     (effects (font (size 1.27 1.27)) (justify right bottom))
   )
-  (label "INJ5" (at 370.84 104.14 180)
+  (label "VVT" (at 372.11 104.14 180)
     (effects (font (size 1.27 1.27)) (justify right bottom))
   )
-  (label "INJ6" (at 370.84 106.68 180)
+  (label "BOOST" (at 372.11 106.68 180)
     (effects (font (size 1.27 1.27)) (justify right bottom))
   )
-  (label "IDLE" (at 370.84 109.22 180)
+  (label "IDLE" (at 372.11 109.22 180)
     (effects (font (size 1.27 1.27)) (justify right bottom))
   )
-  (label "INJ8" (at 370.84 111.76 180)
+  (label "VICS" (at 372.11 111.76 180)
     (effects (font (size 1.27 1.27)) (justify right bottom))
   )
@@
     (effects (font (size 1.27 1.27)) (justify left bottom))
   )
+  (label "EXT_SPI_CS" (at 457.2 78.74 0)
+    (effects (font (size 1.27 1.27)) (justify left bottom))
+  )
   (label "EXT_SPI_CS2" (at 457.2 81.28 0)
     (effects (font (size 1.27 1.27)) (justify left bottom))
@@
     (in_bom yes) (on_board yes) (fields_autoplaced)
     (property "Reference" "M3" (id 0) (at 473.71 215.1338 0))
-    (property "Value" "Module-mcu-0.5" (id 1) (at 473.71 217.4325 0))
+    (property "Value" "Module-mcu144-0.5" (id 1) (at 473.71 217.4325 0))
     (property "Footprint" "hellen-one-mcu-0.3:mcu" (id 2) (at 455.93 218.44 0)
       (effects (font (size 1.27 1.27)) hide)
@@
       (effects (font (size 1.27 1.27)) (justify left))
     )
-    (property "Value" "Module-mcu-0.5" (id 1) (at 418.4651 206.0078 0)
+    (property "Value" "Module-mcu144-0.5" (id 1) (at 418.4651 206.0078 0)
       (effects (font (size 1.27 1.27)) (justify left))
     )
@@
       (effects (font (size 1.27 1.27)) (justify right))
     )
-    (property "Value" "Module-mcu-0.5" (id 1) (at 418.4651 67.5778 0)
+    (property "Value" "Module-mcu144-0.5" (id 1) (at 418.4651 67.5778 0)
       (effects (font (size 1.27 1.27)) (justify right))
     )
@@
   )
   (symbol (lib_id "hellen-one-mcu-0.3:Module-mcu-0.3") (at 435.61 68.58 0) (unit 1)
-    (in_bom yes) (on_board yes) (fields_autoplaced)
+    (in_bom yes) (on_board yes)
     (property "Reference" "M3" (id 0) (at 445.9605 65.2738 0))
-    (property "Value" "Module-mcu-0.5" (id 1) (at 445.9605 67.5725 0))
+    (property "Value" "Module-mcu144-0.5" (id 1) (at 451.0405 67.5725 0))
     (property "Footprint" "hellen-one-mcu-0.3:mcu" (id 2) (at 435.61 68.58 0)
       (effects (font (size 1.27 1.27)) hide)
@@
     )
     (path "/a6bf355d-1d5f-4e79-8e3f-45e3bddf3ceb"
-      (reference "M3") (unit 1) (value "Module-mcu-0.5") (footprint "hellen-one-mcu-0.3:mcu")
+      (reference "M3") (unit 1) (value "Module-mcu144-0.5") (footprint "hellen-one-mcu-0.3:mcu")
     )
     (path "/915d735b-9683-4d94-8b0d-1fa27ebac489"
-      (reference "M3") (unit 2) (value "Module-mcu-0.5") (footprint "hellen-one-mcu-0.3:mcu")
+      (reference "M3") (unit 2) (value "Module-mcu144-0.5") (footprint "hellen-one-mcu-0.3:mcu")
     )
     (path "/5f1c7f30-e456-4e5e-847b-c87579bb1a4c"
-      (reference "M3") (unit 3) (value "Module-mcu-0.5") (footprint "hellen-one-mcu-0.3:mcu")
+      (reference "M3") (unit 3) (value "Module-mcu144-0.5") (footprint "hellen-one-mcu-0.3:mcu")
     )
     (path "/a7d95f89-5755-415c-ab05-3cba0bcc1e6a"
-      (reference "M3") (unit 4) (value "Module-mcu-0.5") (footprint "hellen-one-mcu-0.3:mcu")
+      (reference "M3") (unit 4) (value "Module-mcu144-0.5") (footprint "hellen-one-mcu-0.3:mcu")
     )
     (path "/46c92d79-ab77-4cea-933a-f95fdcee2757"
