File: hellen64_NB1.kicad_sch (KiCad schematic)
At the start: 192 parts, among them J1 USB_B_Mini, J11 Conn_01x01, J13 Conn_01x01, J14 Conn_01x01, J15 Conn_01x01, J16 Conn_01x01, J17 Conn_01x01, J19 Conn_01x01, J2 Conn_01x05_Male, J20 Conn_01x01, J21 Conn_01x01, J22 Conn_01x01, J24 Conn_01x01, J25 AudioJack3_SwitchTR, J27 Conn_01x06, J3 MiniFit, J4 Conn_02x12_Odd_Even, J5 USB_B, J6 ETB, M1 Module-input-0.1, M10 Module-power12-0.2, M11 Module-power5-0.2, M12 Module-wbo-0.3, M13 Module-can-0.1, M2 Module-ign8-0.1, M3 Module-mcu144-0.5, M4 Module-sd-0.1, M5 Module-output-0.3, M6 Module-dinput4-0.1, M7 Module-stlink-0.1, M8 Module-can-0.1, M9 Module-knock-0.1, P1 Pad, P10 Pad, P11 Pad, P12 Pad, P13 Pad, P14 Pad, P15 Pad, P17 Pad, P18 Pad, P19 Pad, P2 178780-1, P20 Pad, P22 Pad, P23 Pad, P24 Pad, P25 Pad, P28 Pad, P29 Pad, P30 Pad, P31 Pad, P32 Pad, P38 Pad, P4 Pad, P43 Pad, P44 Pad, P47 Pad, P48 Pad, P49 Pad, P5 Pad, P50 Pad, P51 Pad, P52 Pad, P53 Pad, P55 Pad, P56 Pad, P6 Pad, P7 Pad, P8 Pad, P9 Pad, U1 LIS2DW12TR, U2 MPX4_MAP, U3 MCP6002-xSN, U4 LPS25HB, U5 L6205PD

Commit message: https://github.com/rusefi/hellen-NB1-issues/issues/25
Parts:
- added C21: 100n, hellen-one-common:C0603, symbol hellen-one-common:Cap
- added R23: 1k, hellen-one-common:R0603, symbol Device:R
Connections:
- net GND: now also C21.1
- net OUT_ALTERNATOR: now also R23.1; no longer R20.1
- new net: C21.2, R20.1, R23.2
Changed lines of the file:
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@@
   (junction (at 144.78 311.15) (diameter 1.016) (color 0 0 0 0))
   (junction (at 147.32 199.39) (diameter 1.016) (color 0 0 0 0))
+  (junction (at 157.48 166.37) (diameter 1.016) (color 0 0 0 0))
   (junction (at 181.61 355.6) (diameter 1.016) (color 0 0 0 0))
   (junction (at 181.61 358.14) (diameter 1.016) (color 0 0 0 0))
@@
     (stroke (width 0) (type solid) (color 0 0 0 0))
   )
-  (wire (pts (xy 132.08 166.37) (xy 266.7 166.37))
+  (wire (pts (xy 132.08 166.37) (xy 157.48 166.37))
     (stroke (width 0) (type solid) (color 0 0 0 0))
   )
@@
     (stroke (width 0) (type solid) (color 0 0 0 0))
   )
+  (wire (pts (xy 157.48 166.37) (xy 161.29 166.37))
+    (stroke (width 0) (type solid) (color 0 0 0 0))
+  )
   (wire (pts (xy 165.1 373.38) (xy 181.61 373.38))
     (stroke (width 0) (type solid) (color 0 0 0 0))
@@
     (stroke (width 0) (type solid) (color 0 0 0 0))
   )
+  (wire (pts (xy 168.91 166.37) (xy 266.7 166.37))
+    (stroke (width 0) (type solid) (color 0 0 0 0))
+  )
   (wire (pts (xy 181.61 353.06) (xy 181.61 355.6))
     (stroke (width 0) (type solid) (color 0 0 0 0))
@@
     (pin "1")
   )
+  (symbol (lib_id "power:GND") (at 157.48 173.99 0) (unit 1)
+    (in_bom yes) (on_board yes)
+    (property "Reference" "#PWR056" (id 0) (at 157.48 180.34 0)
+      (effects (font (size 1.27 1.27)) hide)
+    )
+    (property "Value" "GND" (id 1) (at 157.5308 177.9334 0))
+    (property "Footprint" "" (id 2) (at 157.48 173.99 0)
+      (effects (font (size 1.27 1.27)) hide)
+    )
+    (property "Datasheet" "" (id 3) (at 157.48 173.99 0)
+      (effects (font (size 1.27 1.27)) hide)
+    )
+    (pin "1")
+  )
   (symbol (lib_id "power:GND") (at 181.61 360.68 270) (mirror x) (unit 1)
     (in_bom yes) (on_board yes) (fields_autoplaced)
@@
     (pin "1")
   )
+  (symbol (lib_id "Device:R") (at 165.1 166.37 270) (mirror x) (unit 1)
+    (in_bom yes) (on_board yes)
+    (property "Reference" "R23" (id 0) (at 160.2118 164.858 90))
+    (property "Value" "1k" (id 1) (at 164.8998 166.3245 90))
+    (property "Footprint" "hellen-one-common:R0603" (id 2) (at 165.1 168.148 90)
+      (effects (font (size 1.27 1.27)) hide)
+    )
+    (property "Datasheet" "~" (id 3) (at 165.1 166.37 0)
+      (effects (font (size 1.27 1.27)) hide)
+    )
+    (property "LCSC" "C21190" (id 4) (at 165.1 166.37 0)
+      (effects (font (size 1.27 1.27)) hide)
+    )
+    (pin "1")
+    (pin "2")
+  )
   (symbol (lib_id "Device:R") (at 227.33 383.54 90) (mirror x) (unit 1)
     (in_bom yes) (on_board yes)
@@
     (pin "2")
   )
+  (symbol (lib_id "hellen-one-common:Cap") (at 157.48 170.18 90) (unit 1)
+    (in_bom yes) (on_board yes)
+    (property "Reference" "C21" (id 0) (at 160.2741 169.0306 90)
+      (effects (font (size 1.27 1.27)) (justify right))
+    )
+    (property "Value" "100n" (id 1) (at 160.2741 171.3293 90)
+      (effects (font (size 1.27 1.27)) (justify right))
+    )
+    (property "Footprint" "hellen-one-common:C0603" (id 2) (at 161.29 172.72 0)
+      (effects (font (size 1.27 1.27)) hide)
+    )
+    (property "Datasheet" "" (id 3) (at 157.48 173.99 90)
+      (effects (font (size 1.27 1.27)) hide)
+    )
+    (property "LCSC" "C14663" (id 4) (at 157.48 170.18 0)
+      (effects (font (size 1.27 1.27)) hide)
+    )
+    (pin "1")
+    (pin "2")
+  )
   (symbol (lib_id "hellen-one-common:Cap") (at 184.15 321.31 90) (unit 1)
     (in_bom yes) (on_board yes)
@@
       (reference "#PWR055") (unit 1) (value "+5VA") (footprint "")
     )
+    (path "/f9b5a45a-ab76-4cfd-a506-11d994bd70c5"
+      (reference "#PWR056") (unit 1) (value "GND") (footprint "")
+    )
     (path "/e5f4a915-0042-46bf-9b66-1c48bba43b37"
       (reference "#PWR057") (unit 1) (value "+5VA") (footprint "")
@@
       (reference "C20") (unit 1) (value "10u") (footprint "hellen-one-common:C0805")
     )
+    (path "/755fc5a3-5a1b-43f6-aa19-c36603d0ec11"
+      (reference "C21") (unit 1) (value "100n") (footprint "hellen-one-common:C0603")
+    )
     (path "/ecbba2ec-57c3-41e0-9e70-636da83aa612"
       (reference "D1") (unit 1) (value "LED-GREEN-0805") (footprint "hellen-one-common:LED-0805")
@@
       (reference "R22") (unit 1) (value "Jumper-Pad-Pad") (footprint "hellen-one-common:PAD-0805-PAD")
     )
+    (path "/bd8c17b2-d53d-44b9-8115-2914a71daed2"
+      (reference "R23") (unit 1) (value "1k") (footprint "hellen-one-common:R0603")
+    )
     (path "/2b204e65-1159-43b2-b60a-8f9bea35581e"

Commit message: rev.C https://github.com/rusefi/hellen-NB1-issues/issues/32 https://github.com/rusefi/hellen-NB1-issues/issues/30 https://github.com/rusefi/hellen-NB1-issues/issues/28 https://github.com/rusefi/hellen-NB1-issues/issues/27
Parts:
- added C22: 1u, hellen-one-common:C0603, symbol hellen-one-common:Cap
- added R29: SMD1206B035TF/16, hellen-one-common:R1206, symbol hellen-one-common:Res
- added R41: 4.7k, hellen-one-common:R0603, symbol hellen-one-common:Res
- added U6: TLS115, hellen-one-common:PG-DSO-8-43, symbol hellen-one-common:TLS115
- M3: value Module-mcu144-0.5 -> Module-mcu144-0.6
- R23: value 1k -> 0; LCSC C21190 -> C21189
Connections:
- net +12V: now also U6.8 (IN)
- net +5V: now also R41.1, U6.5 (ADJ), U6.7 (EN)
- net +5VA: now also R29.1; no longer J6.1 (Pin_1), J6.2 (Pin_2), P2.27 (2I), P2.73 (4F)
- net GND: now also C22.1, U6.3 (GND), U6.9 (GND)
- new net: R41.2, U6.4 (PG)
- new net +5VAS: C22.2, J6.1 (Pin_1), J6.2 (Pin_2), P2.27 (2I), P2.73 (4F), R29.2, U6.1 (OUT)
Other:
- note added: "* Warning! Remove R29 is you use TLS115"
- note added: "Protected 5V analog power supply for Sensors"
